File: pmod-sim/tt-audio-pmod.kicad_sch (KiCad schematic)
At the start: 11 parts

Commit message: hella audio testing
Parts:
- removed L2: 150uH, symbol Device:L
- removed PWM1: VPULSE, symbol Simulation_SPICE:VPULSE
- removed R5: 15R, Resistor_SMD:R_0603_1608Metric, symbol Device:R
- added V2: VSIN, symbol Simulation_SPICE:VSIN
- R4: value 200R -> 300R
Connections:
- net GND: now also V2.2
- net Vout: now also C2.1, R3.1
- net vin: now reaches R1.2
- net vin: now also V2.1
- net vout2: now reaches C2.2, C6.1, R2.1, R4.1
Other:
- note added: ".ac dec 100 1 500k"
- note removed: ".tran 1n 50u"
